File: hardware/_autosave-ptSolar.kicad_sch (KiCad schematic)
At the start: 64 parts, among them J4 6 Pin Male Header, J5 Conn_02x04_Odd_Even, Q1 BSS138, Q2 MMBT3904, Q3 BSS138, Q4 BSS138, U1 ATGM336H-5N31, U2 SA818S-V, U5 LP3985IM5-3.3/NOPB, U7 MEGA8-AI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

Commit message: Added Breakout Board for powering and programming the ptSolar.
Parts:
- ANT2b1: footprint Custom DS:Small Test Point Pin -> TestPoint:TestPoint_THTPad_1.5x1.5mm_Drill0.7mm
Changed lines of the file:
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@@
 			)
 		)
-		(property "Footprint" "Custom DS:Small Test Point Pin"
+		(property "Footprint" "TestPoint:TestPoint_THTPad_1.5x1.5mm_Drill0.7mm"
 			(at 351.79 97.79 0)
 			(effects
